File: Antenna-controller.kicad_pcb (KiCad board)
At the start: 2 copper layers, 96.5 x 71.1 mm, 16 parts, among them J1 Power_Supply, J3 SPI_Conn, M1 Motor_DC, Q1 BD138, Q2 BD137, Q3 BD138, Q4 BD137, U1 MCT6, U2 generic_imu, U3 ADG3300

Commit message: idk doing a backup
Parts:
- removed J3: SPI_Conn, Connector_PinHeader_1.00mm:PinHeader_1x05_P1.00mm_Horizontal
- removed R3, R4: R1k, Resistor_THT:R_Axial_DIN0207_L6.3mm_D2.5mm_P10.16mm_Horizontal
- removed U3: ADG3300, ab2_tssop:AB2_TSSOP20
- added J2: SPI_conn, Connector_PinHeader_1.27mm:PinHeader_1x06_P1.27mm_Horizontal, F.Cu at (154.8, 51.9)
- added Q10: fdv303n, Package_TO_SOT_SMD:SOT-23_Handsoldering, B.Cu at (135.9, 57.1)
- added Q5: fdv303n, Package_TO_SOT_SMD:SOT-23_Handsoldering, B.Cu at (148.9, 57.1)
- added Q6: fdv303n, Package_TO_SOT_SMD:SOT-23_Handsoldering, B.Cu at (155.2, 57.1)
- added Q7: fdv303n, Package_TO_SOT_SMD:SOT-23_Handsoldering, B.Cu at (161.3, 57.1)
- added Q8: fdv303n, Package_TO_SOT_SMD:SOT-23_Handsoldering, B.Cu at (167.6, 57.1)
- added Q9: fdv303n, Package_TO_SOT_SMD:SOT-23_Handsoldering, B.Cu at (142.2, 57.1)
- added R10: R10k, Resistor_THT:R_Axial_DIN0207_L6.3mm_D2.5mm_P10.16mm_Horizontal, F.Cu at (167.6, 62.2)
- added R11: R10k, Resistor_THT:R_Axial_DIN0207_L6.3mm_D2.5mm_P10.16mm_Horizontal, F.Cu at (141.0, 62.2)
- added R12: R10k, Resistor_THT:R_Axial_DIN0207_L6.3mm_D2.5mm_P10.16mm_Horizontal, F.Cu at (134.6, 62.2)
- added R13: R10k, Resistor_THT:R_Axial_DIN0207_L6.3mm_D2.5mm_P10.16mm_Horizontal, F.Cu at (123.6, 98.0)
- added R14: R10k, Resistor_THT:R_Axial_DIN0207_L6.3mm_D2.5mm_P10.16mm_Horizontal, F.Cu at (129.8, 98.0)
- added R15: R10k, Resistor_THT:R_Axial_DIN0207_L6.3mm_D2.5mm_P10.16mm_Horizontal, F.Cu at (135.9, 98.0)
- added R16: R10k, Resistor_THT:R_Axial_DIN0207_L6.3mm_D2.5mm_P10.16mm_Horizontal, F.Cu at (167.6, 77.5)
- added R17: R10k, Resistor_THT:R_Axial_DIN0207_L6.3mm_D2.5mm_P10.16mm_Horizontal, F.Cu at (151.1, 76.2)
- added R18: R10k, Resistor_THT:R_Axial_DIN0207_L6.3mm_D2.5mm_P10.16mm_Horizontal, F.Cu at (134.6, 82.5)
- added R7: R10k, Resistor_THT:R_Axial_DIN0207_L6.3mm_D2.5mm_P10.16mm_Horizontal, F.Cu at (148.4, 62.2)
- added R8: R10k, Resistor_THT:R_Axial_DIN0207_L6.3mm_D2.5mm_P10.16mm_Horizontal, F.Cu at (154.9, 62.2)
- added R9: R10k, Resistor_THT:R_Axial_DIN0207_L6.3mm_D2.5mm_P10.16mm_Horizontal, F.Cu at (161.3, 62.2)
- added REF**: MountingHole_2.1mm, MountingHole:MountingHole_2.1mm, F.Cu at (124.5, 49.5)
- added REF**: MountingHole_2.1mm, MountingHole:MountingHole_2.1mm, F.Cu at (124.5, 118.0)
- added REF**: MountingHole_2.1mm, MountingHole:MountingHole_2.1mm, F.Cu at (194.0, 49.5)
- added REF**: MountingHole_2.1mm, MountingHole:MountingHole_2.1mm, F.Cu at (194.0, 118.0)
- added s-lite1: uStepper_s-lite, Connector_PinHeader_1.27mm:PinHeader_1x11_P1.27mm_Horizontal, F.Cu at (190.6, 59.7)
- Q1, Q3: value BD138 -> Q_PMOS_DGS; footprint Package_TO_SOT_THT:TO-126-3_Vertical -> Package_TO_SOT_THT:TO-220-3_Horizontal_TabDown
- Q2, Q4: value BD137 -> Q_NMOS_DGS; footprint Package_TO_SOT_THT:TO-126-3_Vertical -> Package_TO_SOT_THT:TO-251-3-1EP_Horizontal_TabDown
- R1, R2: value R1k -> R
- R5, R6: value R100 -> R190
- U2: footprint Connector_PinHeader_1.27mm:PinHeader_1x08_P1.27mm_Vertical -> Connector_PinHeader_1.27mm:PinHeader_1x08_P1.27mm_Horizontal
- moved J1 175.3 mm to (189.5, 94.3), turned to 90 degrees
- moved M1 174.7 mm to (189.5, 112.0), turned to 90 degrees
- moved Q4 139.9 mm to (178.0, 108.0), turned to 180 degrees
- moved Q2 139.5 mm to (167.3, 108.2), turned to 180 degrees
- moved Q3 135.3 mm to (173.5, 99.2)
- moved Q1 134.0 mm to (162.0, 99.2)
- moved R1 120.7 mm to (154.0, 92.0)
- moved R2 111.0 mm to (143.9, 99.0), turned to 0 degrees
- moved U1 102.2 mm to (139.5, 106.7), turned to 0 degrees
- moved R6 97.0 mm to (134.6, 104.1)
- moved R5 88.5 mm to (128.3, 104.1)
- moved U2 65.4 mm to (135.2, 52.0), turned to 90 degrees
Connections:
- Q1 pad 2: Net-(M1-Pad1) -> forward
- Q1 pad 3: Net-(Q1-Pad3) -> Net-(M1-Pad1)
- Q2 pad 1: GND -> Net-(M1-Pad1)
- Q2 pad 2: Net-(M1-Pad1) -> forward
- Q2 pad 3: Net-(Q2-Pad3) -> GND
- Q3 pad 2: Net-(M1-Pad2) -> rev
- Q3 pad 3: Net-(Q3-Pad3) -> Net-(M1-Pad2)
- Q4 pad 1: GND -> Net-(M1-Pad2)
- Q4 pad 2: Net-(M1-Pad2) -> rev
- Q4 pad 3: Net-(Q4-Pad3) -> GND
- R1 pad 2: Net-(Q1-Pad3) -> GND
- R2 pad 1: forward -> GND
- R2 pad 2: Net-(Q2-Pad3) -> rev
- R5 pad 1: rev_input_3.3V -> rev_input_5V
- R6 pad 1: forward_input_3.3V -> forward_input_5V
Routing:
- net +3V3: track 0.00 -> 160.4 mm
- net imu_scl_5V: track 0.00 -> 143.0 mm
- net imu_sda_5V: track 0.00 -> 136.9 mm
- net SCK_5V: track 0.00 -> 115.8 mm
- net SS1_5V: track 0.00 -> 107.6 mm
- net 5V: track 0.00 -> 96.7 mm
- net MISO_5V: track 0.00 -> 90.5 mm
- net rev_input_5V: track 0.00 -> 77.6 mm
- net forward_input_5V: track 0.00 -> 69.6 mm
- net MOSI_5V: track 0.00 -> 62.8 mm
- net +6V: track 0.00 -> 49.9 mm
- net rev: track 0.00 -> 43.1 mm
- net forward: track 0.00 -> 41.5 mm
- net Net-(M1-Pad1): track 0.00 -> 32.9 mm
- net SS1_3.3V: track 0.00 -> 25.0 mm
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- added copper zone on B.Cu, net GND
Other:
- board size 96.5 x 71.1 mm -> 77.5 x 76.5 mm

Commit message: Update of PCB
Parts:
- J2: footprint Connector_PinHeader_1.27mm:PinHeader_1x06_P1.27mm_Horizontal -> Connector_PinHeader_2.54mm:PinHeader_1x06_P2.54mm_Horizontal
- Q1, Q3: value Q_PMOS_DGS -> SUP75P03-07; footprint Package_TO_SOT_THT:TO-220-3_Horizontal_TabDown -> Package_TO_SOT_THT:TO-220-3_Vertical
- Q2, Q4: value Q_NMOS_DGS -> IRLU024N; footprint Package_TO_SOT_THT:TO-251-3-1EP_Horizontal_TabDown -> Package_TO_SOT_THT:TO-251-3_Vertical
- R1, R2: value R -> 10k
- U2: footprint Connector_PinHeader_1.27mm:PinHeader_1x08_P1.27mm_Horizontal -> Connector_PinHeader_2.54mm:PinHeader_1x08_P2.54mm_Horizontal
- s-lite1: footprint Connector_PinHeader_1.27mm:PinHeader_1x11_P1.27mm_Horizontal -> Connector_PinHeader_2.54mm:PinHeader_1x11_P2.54mm_Horizontal
- moved R2 40.3 mm to (184.2, 102.1), turned to 180 degrees
- moved R15 25.8 mm to (160.3, 89.4), turned to -90 degrees
- moved R1 18.1 mm to (168.7, 102.6)
- moved R16 18.0 mm to (154.2, 89.4), turned to -90 degrees
- moved R12 14.4 mm to (124.7, 72.6)
- moved Q10 14.0 mm to (126.0, 67.1)
- moved R11 13.7 mm to (132.1, 72.6)
- moved R17 13.6 mm to (147.8, 89.4), turned to -90 degrees
- moved Q9 13.3 mm to (133.3, 67.1)
- moved R7 12.9 mm to (140.5, 72.4)
- moved Q5 12.9 mm to (141.0, 67.3)
- moved Q6 12.4 mm to (148.1, 67.3)
- moved R8 12.4 mm to (147.8, 72.4)
- moved Q7 11.5 mm to (156.0, 67.3)
- moved R9 11.5 mm to (156.0, 72.4)
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Connections:
- Q1 pad 1: +6V -> forward
- Q1 pad 2: forward -> +6V
- Q2 pad 1: Net-(M1-Pad1) -> forward
- Q2 pad 2: forward -> Net-(M1-Pad1)
- Q3 pad 1: +6V -> rev
- Q3 pad 2: rev -> +6V
- Q4 pad 1: Net-(M1-Pad2) -> rev
- Q4 pad 2: rev -> Net-(M1-Pad2)
Routing:
- net SS1_5V: track 107.6 -> 59.1 mm
- net imu_scl_5V: track 143.0 -> 96.7 mm
- net +3V3: track 160.4 -> 206.2 mm
- net imu_sda_5V: track 136.9 -> 93.2 mm
- net SCK_5V: track 115.8 -> 87.7 mm
- net MISO_3.3V: track 16.1 -> 34.1 mm
- net imu_scl_3.3V: track 13.3 -> 29.6 mm
- net SCK_3.3V: track 22.8 -> 38.9 mm
- net MOSI_5V: track 62.8 -> 78.6 mm
- net imu_sda_3.3V: track 12.6 -> 27.6 mm
- net MOSI_3.3V: track 17.1 -> 29.8 mm
- net Net-(M1-Pad1): track 32.9 -> 41.3 mm
- net rev_input_5V: track 77.6 -> 69.4 mm
- net MISO_5V: track 90.5 -> 82.8 mm
- net forward: track 41.5 -> 35.0 mm
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