File: Antenna-controller.kicad_sch (KiCad schematic)
At the start: 17 parts, among them J1 Power_Supply, J3 SPI_Conn, M1 Motor_DC, Q1 BD138, Q2 BD137, Q3 BD138, Q4 BD137, U1 MCT6, U2 generic_imu, U3 ADG3300

Commit message: idk doing a backup
Parts:
- removed J3: SPI_Conn, Connector_PinHeader_1.00mm:PinHeader_1x05_P1.00mm_Horizontal, symbol Connector:Conn_01x05_Female
- removed Q1, Q3: BD138, Package_TO_SOT_THT:TO-126-3_Vertical, symbol Transistor_BJT:BD138
- removed Q2, Q4: BD137, Package_TO_SOT_THT:TO-126-3_Vertical, symbol Transistor_BJT:BD137
- removed R1, R2, R3, R4: R1k, Resistor_THT:R_Axial_DIN0207_L6.3mm_D2.5mm_P10.16mm_Horizontal, symbol Device:R
- removed U3: ADG3300, ab2_tssop:AB2_TSSOP20, symbol Logic_LevelTranslator:ADG3300
- added J2: SPI_conn, Connector_PinHeader_1.27mm:PinHeader_1x06_P1.27mm_Horizontal, symbol Connector:Conn_01x06_Female
- added Q10, Q5, Q6, Q7, Q8, Q9: fdv303n, Package_TO_SOT_SMD:SOT-23_Handsoldering, symbol Device:Q_NMOS_GSD
- added Q? (x2): Q_PMOS_DGS, symbol Device:Q_PMOS_DGS
- added Q? (x2): Q_NMOS_DGS, symbol Device:Q_NMOS_DGS
- added R10, R11, R12, R13, R14, R15, R16, R17, R18, R7, R8, R9: R10k, Resistor_THT:R_Axial_DIN0207_L6.3mm_D2.5mm_P10.16mm_Horizontal, symbol Device:R
- added R? (x2): R, symbol Device:R
- R5, R6: value R100 -> R190
- U2: footprint Connector_PinHeader_1.27mm:PinHeader_1x08_P1.27mm_Vertical -> Connector_PinHeader_1.27mm:PinHeader_1x08_P1.27mm_Horizontal
- s-lite1: footprint (none) -> Connector_PinHeader_1.27mm:PinHeader_1x11_P1.27mm_Horizontal
Connections:
- net forward_input_3.3V is gone; now on net forward_input_5V: R6.1
- net rev_input_3.3V is gone; now on net rev_input_5V: R5.1
- net +3V3: now also s-lite1.1 (3.3V), J2.5 (Pin_5), Q10.1 (G), Q5.1 (G), Q6.1 (G), Q7.1 (G), Q8.1 (G), Q9.1 (G), R10.2, R11.2, R12.2, R7.2, R8.2, R9.2; no longer s-lite1.2 (3.3V)
- net +6V: now also Q?.1 (D), Q?.1 (D)
- net 5V: now also s-lite1.2 (5V), R13.2, R14.2, R15.2, R16.2, R17.2, R18.2; no longer s-lite1.3 (5V)
- net GND: now also s-lite1. (VIN), J2.6 (Pin_6), Q?.3 (S), Q?.3 (S), R?.1, R?.2; no longer s-lite1.4 (GND), s-lite1.5 (GND)
- net MISO_3.3V: now also J2.2 (Pin_2), Q6.2 (S), R8.1
- net MISO_5V: now also s-lite1.4 (A1/MISO1), Q6.3 (D), R17.1; no longer s-lite1.15 (D5/MISO0/RX1)
- net MOSI_3.3V: now also J2.3 (Pin_3), Q7.2 (S), R9.1
- net MOSI_5V: now also s-lite1.3 (A0/MOSI1), Q7.3 (D), R16.1; no longer s-lite1.16 (D4/MOSI0/TX1)
- net SCK_3.3V: now also J2.1 (Pin_1), Q5.2 (S), R7.1
- net SCK_5V: now also s-lite1.5 (A2/SCK1), Q5.3 (D), R18.1; no longer s-lite1.14 (D6/SCK0)
- net forward: now also Q?.2 (G), Q?.2 (G), R?.1
- net forward_input_5V: now also s-lite1.10 (D0/RX0); no longer s-lite1.20 (D0/RX0)
- net imu_scl_3.3V: now also Q10.2 (S), R12.1
- net imu_scl_5V: now also s-lite1.8 (A4/SCL0), Q10.3 (D), R13.1; no longer s-lite1.13 (A4/SCL0)
- net imu_sda_3.3V: now also Q9.2 (S), R11.1
- net imu_sda_5V: now also s-lite1.7 (A3/SDA0), Q9.3 (D), R14.1; no longer s-lite1.12 (A3/SDA0)
- net rev: now also Q?.2 (G), Q?.2 (G), R?.2
- net rev_input_5V: now also s-lite1.9 (D1/TX0); no longer s-lite1.19 (D1/TX0)
- net SS1_5V: now reaches s-lite1.6 (AUX1/A5/SS1)
- net SS1_5V: now also Q8.3 (D), R15.1
- net at M1.1 (+): now also Q?.1 (D), Q?.3 (S)
- net at M1.2 (-): now also Q?.1 (D), Q?.3 (S)
- new net SS1_3.3V: J2.4 (Pin_4), Q8.2 (S), R10.1
Other:
- note added: "Logic level converter 5V - 3.3V"
- moved on the sheet: R5, R6, U1, U2

Commit message: Update of PCB
Parts:
- J2: footprint Connector_PinHeader_1.27mm:PinHeader_1x06_P1.27mm_Horizontal -> Connector_PinHeader_2.54mm:PinHeader_1x06_P2.54mm_Horizontal
- Q1, Q3: renamed from Q?; value Q_PMOS_DGS -> (none); symbol Device:Q_PMOS_DGS -> Device:Q_PMOS_GDS
- Q2, Q4: renamed from Q?; value Q_NMOS_DGS -> (none); symbol Device:Q_NMOS_DGS -> Device:Q_NMOS_GDS
- R1, R2: renamed from R?; value R -> (none)
- U2: footprint Connector_PinHeader_1.27mm:PinHeader_1x08_P1.27mm_Horizontal -> Connector_PinHeader_2.54mm:PinHeader_1x08_P2.54mm_Horizontal
- s-lite1: footprint Connector_PinHeader_1.27mm:PinHeader_1x11_P1.27mm_Horizontal -> Connector_PinHeader_2.54mm:PinHeader_1x11_P2.54mm_Horizontal
Connections:
- net +6V: now also Q1.2 (D), Q3.2 (D); no longer Q1.1 (D), Q3.1 (D)
- net forward: now also Q1.1 (G), Q2.1 (G); no longer Q1.2 (G), Q2.2 (G)
- net rev: now also Q3.1 (G), Q4.1 (G); no longer Q3.2 (G), Q4.2 (G)
- net at M1.2 (-), Q3.3 (S): now also Q4.2 (D); no longer Q4.1 (D)
- net at M1.1 (+), Q1.3 (S): now also Q2.2 (D); no longer Q2.1 (D)
Changed lines of the file:
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@@
     (property "Reference" "s-lite1" (id 0) (at 120.65 45.72 0))
     (property "Value" "uStepper_s-lite" (id 1) (at 120.65 48.26 0))
-    (property "Footprint" "Connector_PinHeader_1.27mm:PinHeader_1x11_P1.27mm_Horizontal" (id 2) (at 118.11 60.96 0)
+    (property "Footprint" "Connector_PinHeader_2.54mm:PinHeader_1x11_P2.54mm_Horizontal" (id 2) (at 118.11 60.96 0)
       (effects (font (size 1.27 1.27)) hide)
     )
@@
     (pin "3")
   )
-  (symbol (lib_id "Device:Q_PMOS_DGS") (at 67.31 48.26 0) (mirror y) (unit 1)
-    (in_bom yes) (on_board yes) (fields_autoplaced)
-    (property "Reference" "Q?" (id 0) (at 60.96 46.9899 0)
-      (effects (font (size 1.27 1.27)) (justify left))
-    )
-    (property "Value" "Q_PMOS_DGS" (id 1) (at 60.96 49.5299 0)
+  (symbol (lib_id "Device:Q_PMOS_GDS") (at 67.31 48.26 0) (mirror y) (unit 1)
+    (in_bom yes) (on_board yes)
+    (property "Reference" "Q3" (id 0) (at 60.96 46.9899 0)
+      (effects (font (size 1.27 1.27)) (justify left))
+    )
+    (property "Value" "" (id 1) (at 71.12 54.61 0)
       (effects (font (size 1.27 1.27)) (justify left))
     )
@@
       (effects (font (size 1.27 1.27)) (justify left))
     )
-    (property "Footprint" "Connector_PinHeader_1.27mm:PinHeader_1x06_P1.27mm_Horizontal" (id 2) (at 143.51 29.845 0)
+    (property "Footprint" "Connector_PinHeader_2.54mm:PinHeader_1x06_P2.54mm_Horizontal" (id 2) (at 143.51 29.845 0)
       (effects (font (size 1.27 1.27)) hide)
     )
@@
   )
   (symbol (lib_id "Device:R") (at 38.1 73.66 90) (mirror x) (unit 1)
-    (in_bom yes) (on_board yes) (fields_autoplaced)
-    (property "Reference" "R?" (id 0) (at 38.1 67.31 90))
-    (property "Value" "R" (id 1) (at 38.1 69.85 90))
+    (in_bom yes) (on_board yes)
+    (property "Reference" "R1" (id 0) (at 38.1 71.12 90))
+    (property "Value" "" (id 1) (at 38.1 76.2 90))
     (property "Footprint" "" (id 2) (at 38.1 71.882 90)
       (effects (font (size 1.27 1.27)) hide)
@@
     (pin "1")
   )
-  (symbol (lib_id "Device:Q_NMOS_DGS") (at 67.31 68.58 0) (mirror y) (unit 1)
-    (in_bom yes) (on_board yes) (fields_autoplaced)
-    (property "Reference" "Q?" (id 0) (at 60.96 67.3099 0)
-      (effects (font (size 1.27 1.27)) (justify left))
-    )
-    (property "Value" "Q_NMOS_DGS" (id 1) (at 60.96 69.8499 0)
+  (symbol (lib_id "Device:Q_NMOS_GDS") (at 67.31 68.58 0) (mirror y) (unit 1)
+    (in_bom yes) (on_board yes)
+    (property "Reference" "Q4" (id 0) (at 60.96 67.3099 0)
+      (effects (font (size 1.27 1.27)) (justify left))
+    )
+    (property "Value" "" (id 1) (at 71.12 63.5 0)
       (effects (font (size 1.27 1.27)) (justify left))
     )
@@
     (pin "3")
   )
-  (symbol (lib_id "Device:Q_PMOS_DGS") (at 39.37 48.26 0) (unit 1)
-    (in_bom yes) (on_board yes) (fields_autoplaced)
-    (property "Reference" "Q?" (id 0) (at 45.72 46.9899 0)
-      (effects (font (size 1.27 1.27)) (justify left))
-    )
-    (property "Value" "Q_PMOS_DGS" (id 1) (at 45.72 49.5299 0)
+  (symbol (lib_id "Device:Q_PMOS_GDS") (at 39.37 48.26 0) (unit 1)
+    (in_bom yes) (on_board yes)
+    (property "Reference" "Q1" (id 0) (at 45.72 46.9899 0)
+      (effects (font (size 1.27 1.27)) (justify left))
+    )
+    (property "Value" "" (id 1) (at 36.83 54.61 0)
       (effects (font (size 1.27 1.27)) (justify left))
     )
@@
   )
   (symbol (lib_id "Device:R") (at 68.58 73.66 90) (unit 1)
-    (in_bom yes) (on_board yes) (fields_autoplaced)
-    (property "Reference" "R?" (id 0) (at 68.58 67.31 90))
-    (property "Value" "R" (id 1) (at 68.58 69.85 90))
+    (in_bom yes) (on_board yes)
+    (property "Reference" "R2" (id 0) (at 68.58 71.12 90))
+    (property "Value" "" (id 1) (at 68.58 76.2 90))
     (property "Footprint" "" (id 2) (at 68.58 75.438 90)
       (effects (font (size 1.27 1.27)) hide)
@@
     (pin "2")
   )
-  (symbol (lib_id "Device:Q_NMOS_DGS") (at 39.37 68.58 0) (unit 1)
-    (in_bom yes) (on_board yes) (fields_autoplaced)
-    (property "Reference" "Q?" (id 0) (at 45.72 67.3099 0)
-      (effects (font (size 1.27 1.27)) (justify left))
-    )
-    (property "Value" "Q_NMOS_DGS" (id 1) (at 45.72 69.8499 0)
+  (symbol (lib_id "Device:Q_NMOS_GDS") (at 39.37 68.58 0) (unit 1)
+    (in_bom yes) (on_board yes)
+    (property "Reference" "Q2" (id 0) (at 45.72 67.3099 0)
+      (effects (font (size 1.27 1.27)) (justify left))
+    )
+    (property "Value" "" (id 1) (at 35.56 63.5 0)
       (effects (font (size 1.27 1.27)) (justify left))
     )
@@
     (property "Reference" "U2" (id 0) (at 98.425 13.97 0))
     (property "Value" "generic_imu" (id 1) (at 98.425 16.51 0))
-    (property "Footprint" "Connector_PinHeader_1.27mm:PinHeader_1x08_P1.27mm_Horizontal" (id 2) (at 97.155 25.4 0)
+    (property "Footprint" "Connector_PinHeader_2.54mm:PinHeader_1x08_P2.54mm_Horizontal" (id 2) (at 97.155 25.4 0)
       (effects (font (size 1.27 1.27)) hide)
     )
@@
     )
     (path "/4969ff4a-6490-4de0-b443-13ef0bc8e284"
-      (reference "J2") (unit 1) (value "SPI_conn") (footprint "Connector_PinHeader_1.27mm:PinHeader_1x06_P1.27mm_Horizontal")
+      (reference "J2") (unit 1) (value "SPI_conn") (footprint "Connector_PinHeader_2.54mm:PinHeader_1x06_P2.54mm_Horizontal")
     )
     (path "/cc28f8de-3b73-48c3-b866-55205e3aa0cb"
       (reference "M1") (unit 1) (value "Motor_DC") (footprint "TerminalBlock:TerminalBlock_Altech_AK300-2_P5.00mm")
     )
+    (path "/802f8b9d-2da3-4d18-84be-eee030f1b7c7"
+      (reference "Q1") (unit 1) (value "SUP75P03-07") (footprint "Package_TO_SOT_THT:TO-220-3_Vertical")
+    )
+    (path "/c3fe8e98-c741-42b2-bffd-809b9acb0d42"
+      (reference "Q2") (unit 1) (value "IRLU024N") (footprint "Package_TO_SOT_THT:TO-251-3_Vertical")
+    )
+    (path "/2b6dba3c-3559-46ff-a0bf-3e295b312c80"
+      (reference "Q3") (unit 1) (value "SUP75P03-07") (footprint "Package_TO_SOT_THT:TO-220-3_Vertical")
+    )
+    (path "/7814eec3-cc1f-43d6-8519-0141d3a94685"
+      (reference "Q4") (unit 1) (value "IRLU024N") (footprint "Package_TO_SOT_THT:TO-251-3_Vertical")
+    )
     (path "/a1d1b2fd-d4b6-4500-8fd3-f0b1d46c735b"
       (reference "Q5") (unit 1) (value "fdv303n") (footprint "Package_TO_SOT_SMD:SOT-23_Handsoldering")
@@
       (reference "Q10") (unit 1) (value "fdv303n") (footprint "Package_TO_SOT_SMD:SOT-23_Handsoldering")
     )
-    (path "/2b6dba3c-3559-46ff-a0bf-3e295b312c80"
-      (reference "Q?") (unit 1) (value "Q_PMOS_DGS") (footprint "")
-    )
-    (path "/7814eec3-cc1f-43d6-8519-0141d3a94685"
-      (reference "Q?") (unit 1) (value "Q_NMOS_DGS") (footprint "")
-    )
-    (path "/802f8b9d-2da3-4d18-84be-eee030f1b7c7"
-      (reference "Q?") (unit 1) (value "Q_PMOS_DGS") (footprint "")
-    )
-    (path "/c3fe8e98-c741-42b2-bffd-809b9acb0d42"
-      (reference "Q?") (unit 1) (value "Q_NMOS_DGS") (footprint "")
+    (path "/52dbbd74-0890-448b-adf7-19ff34fb6f36"
+      (reference "R1") (unit 1) (value "10k") (footprint "Resistor_THT:R_Axial_DIN0207_L6.3mm_D2.5mm_P10.16mm_Horizontal")
+    )
+    (path "/a2dec537-a358-4c00-9961-d77ef5653950"
+      (reference "R2") (unit 1) (value "10k") (footprint "Resistor_THT:R_Axial_DIN0207_L6.3mm_D2.5mm_P10.16mm_Horizontal")
     )
     (path "/6d80a2e4-617a-4bc8-b13f-c3195f583107"
@@
       (reference "R18") (unit 1) (value "R10k") (footprint "Resistor_THT:R_Axial_DIN0207_L6.3mm_D2.5mm_P10.16mm_Horizontal")
     )
-    (path "/52dbbd74-0890-448b-adf7-19ff34fb6f36"
-      (reference "R?") (unit 1) (value "R") (footprint "")
-    )
-    (path "/a2dec537-a358-4c00-9961-d77ef5653950"
-      (reference "R?") (unit 1) (value "R") (footprint "")
-    )
     (path "/2128cd6a-874b-4c20-bf4b-b5c19d67d488"
       (reference "U1") (unit 1) (value "MCT6") (footprint "Package_DIP:DIP-8_W10.16mm_LongPads")
     )
     (path "/c7ceb4fb-e7cc-4b4f-8f48-b50c896daf50"
-      (reference "U2") (unit 1) (value "generic_imu") (footprint "Connector_PinHeader_1.27mm:PinHeader_1x08_P1.27mm_Horizontal")
+      (reference "U2") (unit 1) (value "generic_imu") (footprint "Connector_PinHeader_2.54mm:PinHeader_1x08_P2.54mm_Horizontal")
     )
     (path "/122477c2-4188-45a1-99cd-35320f27efc7"
-      (reference "s-lite1") (unit 1) (value "uStepper_s-lite") (footprint "Connector_PinHeader_1.27mm:PinHeader_1x11_P1.27mm_Horizontal")
-    )
-  )
+      (reference "s-lite1") (unit 1) (value "uStepper_s-lite") (footprint "Connector_PinHeader_2.54mm:PinHeader_1x11_P2.54mm_Horizontal")
+    )
+  )
